Commit message: Fix mesh scaling.
Model looks ok in gazebo now :)

File: urdf/shadowhand.urdf (robot description, URDF)
Before this commit: robot shadowhand, 35 links, 34 joints
Links:
- link ffknuckle: geometry collision box size=0.005 0.005 0.005; visual mesh filename=package://sr_grasp_description/meshes/knuckle.dae scale=0.1 0.1 0.1
- link ffproximal: geometry collision box size=0.008 0.008 0.04; visual mesh filename=package://sr_grasp_description/meshes/F3.dae scale=0.1 0.1 0.1
- link forearm: geometry collision cylinder length=0.180 radius=0.06; visual mesh filename=package://sr_grasp_description/meshes/forearm.dae scale=0.1 0.1 0.1
- link lfknuckle: geometry collision box size=0.005 0.005 0.005; visual mesh filename=package://sr_grasp_description/meshes/knuckle.dae scale=0.1 0.1 0.1
- link lfmetacarpal: geometry collision box size=0.008 0.008 0.03; visual mesh filename=package://sr_grasp_description/meshes/lfmetacarpal.dae scale=0.1 0.1 0.1
- link lfproximal: geometry collision box size=0.008 0.008 0.04; visual mesh filename=package://sr_grasp_description/meshes/F3.dae scale=0.1 0.1 0.1
- link mfknuckle: geometry collision box size=0.005 0.005 0.005; visual mesh filename=package://sr_grasp_description/meshes/knuckle.dae scale=0.1 0.1 0.1
- link mfproximal: geometry collision box size=0.008 0.008 0.04; visual mesh filename=package://sr_grasp_description/meshes/F3.dae scale=0.1 0.1 0.1
- link palm: geometry collision box size=0.05 0.02 0.07; visual mesh filename=package://sr_grasp_description/meshes/palm.dae scale=0.1 0.1 0.1
- link rfknuckle: geometry collision box size=0.005 0.005 0.005; visual mesh filename=package://sr_grasp_description/meshes/knuckle.dae scale=0.1 0.1 0.1
- link rfproximal: geometry collision box size=0.008 0.008 0.04; visual mesh filename=package://sr_grasp_description/meshes/F3.dae scale=0.1 0.1 0.1
- link thproximal: geometry collision box size=0.008 0.008 0.020; visual mesh filename=package://sr_grasp_description/meshes/TH3_z.dae scale=0.1 0.1 0.1
- link wrist: geometry collision box size=0.02 0.02 0.02; visual mesh filename=package://sr_grasp_description/meshes/wrist.dae scale=0.1 0.1 0.1

Commit message: ellipsoid finger tips

File: urdf/shadowhand.urdf (robot description, URDF)
Before this commit: robot shadowhand, 35 links, 34 joints
Links:
- removed link ff_J1_dummy
- removed link ffadapter
- removed link ffbiotac
- removed link lf_J1_dummy
- removed link lfadapter
- removed link lfbiotac
- removed link mf_J1_dummy
- removed link mfadapter
- removed link mfbiotac
- removed link rf_J1_dummy
- removed link rfadapter
- removed link rfbiotac
- removed link thbiotac
- removed link thbiotac_J1_dummy
- added link ffdistal, mass 0.010; collision mesh filename=package://sr_grasp_description/meshes/distal_ellipsoid.dae scale=0.1 0.1 0.1; visual mesh filename=package://sr_grasp_description/meshes/distal_ellipsoid.dae scale=0.1 0.1 0.1
- added link ffmiddle, mass 0.012; collision box size=0.008 0.008 0.015; visual mesh filename=package://sr_grasp_description/meshes/F2.dae scale=0.1 0.1 0.1
- added link lfdistal, mass 0.010; collision mesh filename=package://sr_grasp_description/meshes/distal_ellipsoid.dae scale=0.1 0.1 0.1; visual mesh filename=package://sr_grasp_description/meshes/distal_ellipsoid.dae scale=0.1 0.1 0.1
- added link lfmiddle, mass 0.012; collision box size=0.008 0.008 0.015; visual mesh filename=package://sr_grasp_description/meshes/F2.dae scale=0.1 0.1 0.1
- added link mfdistal, mass 0.010; collision mesh filename=package://sr_grasp_description/meshes/distal_ellipsoid.dae scale=0.1 0.1 0.1; visual mesh filename=package://sr_grasp_description/meshes/distal_ellipsoid.dae scale=0.1 0.1 0.1
- added link mfmiddle, mass 0.012; collision box size=0.008 0.008 0.015; visual mesh filename=package://sr_grasp_description/meshes/F2.dae scale=0.1 0.1 0.1
- added link rfdistal, mass 0.010; collision mesh filename=package://sr_grasp_description/meshes/distal_ellipsoid.dae scale=0.1 0.1 0.1; visual mesh filename=package://sr_grasp_description/meshes/distal_ellipsoid.dae scale=0.1 0.1 0.1
- added link rfmiddle, mass 0.012; collision box size=0.008 0.008 0.015; visual mesh filename=package://sr_grasp_description/meshes/F2.dae scale=0.1 0.1 0.1
- added link thdistal, mass 0.016; collision mesh filename=package://sr_grasp_description/meshes/distal_ellipsoid.dae scale=0.1 0.1 0.1; visual mesh filename=package://sr_grasp_description/meshes/distal_ellipsoid.dae scale=0.1 0.1 0.1
- link fftip: geometry 
- link lftip: geometry 
- link mftip: geometry 
- link rftip: geometry 
- link thmiddle: geometry collision box size=0.008 0.008 0.015; visual mesh filename=package://sr_grasp_description/meshes/TH2_z.dae scale=0.1 0.1 0.1
- link thtip: geometry 
Joints:
- removed joint FF_biotac_joint
- removed joint LF_biotac_joint
- removed joint MF_biotac_joint
- removed joint RF_biotac_joint
- removed joint fftip_fixed_joint
- removed joint lftip_fixed_joint
- removed joint mftip_fixed_joint
- removed joint rftip_fixed_joint
- removed joint th_biotac_joint
- added joint FFtip: type fixed, parent ffdistal, child fftip, origin xyz=0 0 0.026 rpy=0 0 0
- added joint LFtip: type fixed, parent lfdistal, child lftip, origin xyz=0 0 0.026 rpy=0 0 0
- added joint MFtip: type fixed, parent mfdistal, child mftip, origin xyz=0 0 0.026 rpy=0 0 0
- added joint RFtip: type fixed, parent rfdistal, child rftip, origin xyz=0 0 0.026 rpy=0 0 0
- joint FFJ1: child ff_J1_dummy -> ffdistal; limit lower=0.349065850399 upper=0.350811179651 effort=10 velocity=0.1 -> lower=0 upper=1.57079632679 effort=10 velocity=1.0; origin xyz=0 0 0.02 rpy=0 0 0 -> xyz=0 0 0.025 rpy=0 0 0; parent ffadapter -> ffmiddle
- joint FFJ2: child ffadapter -> ffmiddle
- joint LFJ1: child lf_J1_dummy -> lfdistal; limit lower=0.349065850399 upper=0.350811179651 effort=10 velocity=0.1 -> lower=0 upper=1.57079632679 effort=10 velocity=1.0; origin xyz=0 0 0.02 rpy=0 0 0 -> xyz=0 0 0.025 rpy=0 0 0; parent lfadapter -> lfmiddle
- joint LFJ2: child lfadapter -> lfmiddle
- joint MFJ1: child mf_J1_dummy -> mfdistal; limit lower=0.349065850399 upper=0.350811179651 effort=10 velocity=0.1 -> lower=0 upper=1.57079632679 effort=10 velocity=1.0; origin xyz=0 0 0.02 rpy=0 0 0 -> xyz=0 0 0.025 rpy=0 0 0; parent mfadapter -> mfmiddle
- joint MFJ2: child mfadapter -> mfmiddle
- joint RFJ1: child rf_J1_dummy -> rfdistal; limit lower=0.349065850399 upper=0.350811179651 effort=10 velocity=0.1 -> lower=0 upper=1.57079632679 effort=10 velocity=1.0; origin xyz=0 0 0.02 rpy=0 0 0 -> xyz=0 0 0.025 rpy=0 0 0; parent rfadapter -> rfmiddle
- joint RFJ2: child rfadapter -> rfmiddle
- joint THJ1: child thbiotac_J1_dummy -> thdistal; limit lower=0.349065850399 upper=0.350811179651 effort=10 velocity=0.1 -> lower=0 upper=1.571 effort=10 velocity=1.0; origin xyz=0 0 0.02 rpy=0 0 0 -> xyz=0 0 0.032 rpy=0 0 -1.570796327
- joint THJ2: origin xyz=0 0 0.01 rpy=0 0 0 -> xyz=0 0 0 rpy=0 0 0
- joint thtip: origin xyz=-0.009 0.0 0.054 rpy=0 0 -1.571 -> xyz=0 0 0.0275 rpy=0 0 0; parent thmiddle -> thdistal
