Commit message: Re-add the fixed world link.

File: urdf/gazebo_shadowhand_standalone.urdf.xacro (robot description, xacro)
@@ -6,12 +6,9 @@
   </gazebo>
   <!-- adding fixed link to world for the hand not to fall -->
-  <!-- wtf! this crashes when launching but works ok in the dms_gazebo launch. Why? -->
-  <!--
   <link name="world"/>
   <joint name="fixed" type="fixed">
     <parent link="world"/>
-    <child link="base_link"/>
+    <child link="forearm"/>
   </joint>
-  -->
   <!-- loading the shadow hand -->
   <xacro:include filename="$(find sr_grasp_description)/urdf/shadowhand.urdf" />

Commit message: Add wrist transmissions.

File: urdf/gazebo_shadowhand_standalone.urdf.xacro (robot description, xacro)
@@ -5,4 +5,20 @@
     </plugin>
   </gazebo>
+  <transmission name="trans_WRJ1">
+    <type>transmission_interface/SimpleTransmission</type>
+    <joint name="WRJ1"/>
+    <actuator name="motor_WRJ1">
+      <hardwareInterface>EffortJointInterface</hardwareInterface>
+      <mechanicalReduction>1</mechanicalReduction>
+    </actuator>
+  </transmission>
+  <transmission name="trans_WRJ2">
+    <type>transmission_interface/SimpleTransmission</type>
+    <joint name="WRJ2"/>
+    <actuator name="motor_WRJ2">
+      <hardwareInterface>EffortJointInterface</hardwareInterface>
+      <mechanicalReduction>1</mechanicalReduction>
+    </actuator>
+  </transmission>
   <!-- adding fixed link to world for the hand not to fall -->
   <link name="world"/>

Commit message: FF control.

File: urdf/gazebo_shadowhand_standalone.urdf.xacro (robot description, xacro)
@@ -21,4 +21,36 @@
     </actuator>
   </transmission>
+  <transmission name="trans_ffj1">
+    <type>transmission_interface/SimpleTransmission</type>
+    <joint name="FFJ1"/>
+    <actuator name="motor_ffj1">
+      <hardwareInterface>EffortJointInterface</hardwareInterface>
+      <mechanicalReduction>1</mechanicalReduction>
+    </actuator>
+  </transmission>
+  <transmission name="trans_ffj2">
+    <type>transmission_interface/SimpleTransmission</type>
+    <joint name="FFJ2"/>
+    <actuator name="motor_ffj2">
+      <hardwareInterface>EffortJointInterface</hardwareInterface>
+      <mechanicalReduction>1</mechanicalReduction>
+    </actuator>
+  </transmission>
+  <transmission name="trans_ffj3">
+    <type>transmission_interface/SimpleTransmission</type>
+    <joint name="FFJ3"/>
+    <actuator name="motor_ffj3">
+      <hardwareInterface>EffortJointInterface</hardwareInterface>
+      <mechanicalReduction>1</mechanicalReduction>
+    </actuator>
+  </transmission>
+  <transmission name="trans_ffj4">
+    <type>transmission_interface/SimpleTransmission</type>
+    <joint name="FFJ4"/>
+    <actuator name="motor_ffj4">
+      <hardwareInterface>EffortJointInterface</hardwareInterface>
+      <mechanicalReduction>1</mechanicalReduction>
+    </actuator>
+  </transmission>
   <!-- adding fixed link to world for the hand not to fall -->
   <link name="world"/>

Commit message: Add all the other joints.

File: urdf/gazebo_shadowhand_standalone.urdf.xacro (robot description, xacro)
@@ -53,4 +53,132 @@
     </actuator>
   </transmission>
+  <transmission name="trans_mfj1">
+    <type>transmission_interface/SimpleTransmission</type>
+    <joint name="MFJ1"/>
+    <actuator name="motor_mfj1">
+      <hardwareInterface>EffortJointInterface</hardwareInterface>
+      <mechanicalReduction>1</mechanicalReduction>
+    </actuator>
+  </transmission>
+  <transmission name="trans_mfj2">
+    <type>transmission_interface/SimpleTransmission</type>
+    <joint name="MFJ2"/>
+    <actuator name="motor_mfj2">
+      <hardwareInterface>EffortJointInterface</hardwareInterface>
+      <mechanicalReduction>1</mechanicalReduction>
+    </actuator>
+  </transmission>
+  <transmission name="trans_mfj3">
+    <type>transmission_interface/SimpleTransmission</type>
+    <joint name="MFJ3"/>
+    <actuator name="motor_mfj3">
+      <hardwareInterface>EffortJointInterface</hardwareInterface>
+      <mechanicalReduction>1</mechanicalReduction>
+    </actuator>
+  </transmission>
+  <transmission name="trans_mfj4">
+    <type>transmission_interface/SimpleTransmission</type>
+    <joint name="MFJ4"/>
+    <actuator name="motor_mfj4">
+      <hardwareInterface>EffortJointInterface</hardwareInterface>
+      <mechanicalReduction>1</mechanicalReduction>
+    </actuator>
+  </transmission>
+  <transmission name="trans_rfj1">
+    <type>transmission_interface/SimpleTransmission</type>
+    <joint name="RFJ1"/>
+    <actuator name="motor_rfj1">
+      <hardwareInterface>EffortJointInterface</hardwareInterface>
+      <mechanicalReduction>1</mechanicalReduction>
+    </actuator>
+  </transmission>
+  <transmission name="trans_rfj2">
+    <type>transmission_interface/SimpleTransmission</type>
+    <joint name="RFJ2"/>
+    <actuator name="motor_rfj2">
+      <hardwareInterface>EffortJointInterface</hardwareInterface>
+      <mechanicalReduction>1</mechanicalReduction>
+    </actuator>
+  </transmission>
+  <transmission name="trans_rfj3">
+    <type>transmission_interface/SimpleTransmission</type>
+    <joint name="RFJ3"/>
+    <actuator name="motor_rfj3">
+      <hardwareInterface>EffortJointInterface</hardwareInterface>
+      <mechanicalReduction>1</mechanicalReduction>
+    </actuator>
+  </transmission>
+  <transmission name="trans_rfj4">
+    <type>transmission_interface/SimpleTransmission</type>
+    <joint name="RFJ4"/>
+    <actuator name="motor_rfj4">
+      <hardwareInterface>EffortJointInterface</hardwareInterface>
+      <mechanicalReduction>1</mechanicalReduction>
+    </actuator>
+  </transmission>
+  <transmission name="trans_lfj1">
+    <type>transmission_interface/SimpleTransmission</type>
+    <joint name="LFJ1"/>
+    <actuator name="motor_lfj1">
+      <hardwareInterface>EffortJointInterface</hardwareInterface>
+      <mechanicalReduction>1</mechanicalReduction>
+    </actuator>
+  </transmission>
+  <transmission name="trans_lfj2">
+    <type>transmission_interface/SimpleTransmission</type>
+    <joint name="LFJ2"/>
+    <actuator name="motor_lfj2">
+      <hardwareInterface>EffortJointInterface</hardwareInterface>
+      <mechanicalReduction>1</mechanicalReduction>
+    </actuator>
+  </transmission>
+  <transmission name="trans_lfj3">
+    <type>transmission_interface/SimpleTransmission</type>
+    <joint name="LFJ3"/>
+    <actuator name="motor_lfj3">
+      <hardwareInterface>EffortJointInterface</hardwareInterface>
+      <mechanicalReduction>1</mechanicalReduction>
+    </actuator>
+  </transmission>
+  <transmission name="trans_lfj4">
+    <type>transmission_interface/SimpleTransmission</type>
+    <joint name="LFJ4"/>
+    <actuator name="motor_lfj4">
+      <hardwareInterface>EffortJointInterface</hardwareInterface>
+      <mechanicalReduction>1</mechanicalReduction>
+    </actuator>
+  </transmission>
+  <transmission name="trans_thj1">
+    <type>transmission_interface/SimpleTransmission</type>
+    <joint name="THJ1"/>
+    <actuator name="motor_thj1">
+      <hardwareInterface>EffortJointInterface</hardwareInterface>
+      <mechanicalReduction>1</mechanicalReduction>
+    </actuator>
+  </transmission>
+  <transmission name="trans_thj2">
+    <type>transmission_interface/SimpleTransmission</type>
+    <joint name="THJ2"/>
+    <actuator name="motor_thj2">
+      <hardwareInterface>EffortJointInterface</hardwareInterface>
+      <mechanicalReduction>1</mechanicalReduction>
+    </actuator>
+  </transmission>
+  <transmission name="trans_thj3">
+    <type>transmission_interface/SimpleTransmission</type>
+    <joint name="THJ3"/>
+    <actuator name="motor_thj3">
+      <hardwareInterface>EffortJointInterface</hardwareInterface>
+      <mechanicalReduction>1</mechanicalReduction>
+    </actuator>
+  </transmission>
+  <transmission name="trans_thj4">
+    <type>transmission_interface/SimpleTransmission</type>
+    <joint name="THJ4"/>
+    <actuator name="motor_thj4">
+      <hardwareInterface>EffortJointInterface</hardwareInterface>
+      <mechanicalReduction>1</mechanicalReduction>
+    </actuator>
+  </transmission>
   <!-- adding fixed link to world for the hand not to fall -->
   <link name="world"/>

Commit message: Increase effort limits.
Also move the gazebo tags into the gazebo file, leaving shadowhand.urdf to be
just what comes out of running fix_urdf.py

File: urdf/gazebo_shadowhand_standalone.urdf.xacro (robot description, xacro)
@@ -4,4 +4,59 @@
       <robotNamespace>/sh</robotNamespace>
     </plugin>
+  </gazebo>
+  <gazebo reference="ffdistal">
+    <sensor type="contact" name="ffdistal_contact" >
+      <plugin name="ffdistal_gazebo_ros_bumper_controller" filename="libgazebo_ros_bumper.so">
+	<alwaysOn>true</alwaysOn>
+	<updateRate>100.0</updateRate>
+	<frameName>ffdistal</frameName>
+	<bumperTopicName>/sh/contacts/ffdistal</bumperTopicName>
+      </plugin>
+    </sensor>
+    <material>Gazebo/Orange</material>
+  </gazebo>
+  <gazebo reference="mfdistal">
+    <sensor type="contact" name="mf_contact" >
+      <plugin name="mf_gazebo_ros_bumper_controller" filename="libgazebo_ros_bumper.so">
+	<alwaysOn>true</alwaysOn>
+	<updateRate>100.0</updateRate>
+	<frameName>mfdistal</frameName>
+	<bumperTopicName>/sh/contacts/mf</bumperTopicName>
+      </plugin>
+    </sensor>
+    <material>Gazebo/Orange</material>
+  </gazebo>
+  <gazebo reference="rfdistal">
+    <sensor type="contact" name="mf_contact" >
+      <plugin name="mf_gazebo_ros_bumper_controller" filename="libgazebo_ros_bumper.so">
+	<alwaysOn>true</alwaysOn>
+	<updateRate>100.0</updateRate>
+	<frameName>rfdistal</frameName>
+	<bumperTopicName>/sh/contacts/mf</bumperTopicName>
+      </plugin>
+    </sensor>
+    <material>Gazebo/Orange</material>
+  </gazebo>
+  <gazebo reference="lfdistal">
+    <sensor type="contact" name="lf_contact" >
+      <plugin name="lf_gazebo_ros_bumper_controller" filename="libgazebo_ros_bumper.so">
+	<alwaysOn>true</alwaysOn>
+	<updateRate>100.0</updateRate>
+	<frameName>lfdistal</frameName>
+	<bumperTopicName>/sh/contacts/lf</bumperTopicName>
+      </plugin>
+    </sensor>
+    <material>Gazebo/Orange</material>
+  </gazebo>
+  <gazebo reference="thdistal">
+    <sensor type="contact" name="th_contact" >
+      <plugin name="th_gazebo_ros_bumper_controller" filename="libgazebo_ros_bumper.so">
+	<alwaysOn>true</alwaysOn>
+	<updateRate>100.0</updateRate>
+	<frameName>thdistal</frameName>
+	<bumperTopicName>/sh/contacts/th</bumperTopicName>
+      </plugin>
+    </sensor>
+    <material>Gazebo/Orange</material>
   </gazebo>
   <transmission name="trans_wrj1">

File: urdf/shadowhand.urdf (robot description, URDF)
Before this commit: robot shadowhand, 30 links, 29 joints
Joints:
- joint FFJ1: limit lower=0 upper=1.57079632679 effort=10 velocity=1.0 -> lower=0 upper=1.57079632679 effort=100 velocity=1.0
- joint FFJ2: limit lower=0 upper=1.57079632679 effort=10 velocity=1.0 -> lower=0 upper=1.57079632679 effort=100 velocity=1.0
- joint FFJ3: limit lower=0 upper=1.57079632679 effort=10 velocity=1.0 -> lower=0 upper=1.57079632679 effort=100 velocity=1.0
- joint FFJ4: limit lower=-0.43633231299858238 upper=0.43633231299858238 effort=10 velocity=1.0 -> lower=-0.43633231299858238 upper=0.43633231299858238 effort=100 velocity=1.0
- joint LFJ1: limit lower=0 upper=1.57079632679 effort=10 velocity=1.0 -> lower=0 upper=1.57079632679 effort=100 velocity=1.0
- joint LFJ2: limit lower=0 upper=1.57079632679 effort=10 velocity=1.0 -> lower=0 upper=1.57079632679 effort=100 velocity=1.0
- joint LFJ3: limit lower=0 upper=1.57079632679 effort=10 velocity=1.0 -> lower=0 upper=1.57079632679 effort=100 velocity=1.0
- joint LFJ4: limit lower=-0.43633231299858238 upper=0.43633231299858238 effort=10 velocity=1.0 -> lower=-0.43633231299858238 upper=0.43633231299858238 effort=100 velocity=1.0
- joint LFJ5: limit lower=0 upper=0.69813170079773179 effort=10 velocity=1.0 -> lower=0 upper=0.69813170079773179 effort=100 velocity=1.0
- joint MFJ1: limit lower=0 upper=1.57079632679 effort=10 velocity=1.0 -> lower=0 upper=1.57079632679 effort=100 velocity=1.0
- joint MFJ2: limit lower=0 upper=1.57079632679 effort=10 velocity=1.0 -> lower=0 upper=1.57079632679 effort=100 velocity=1.0
- joint MFJ3: limit lower=0 upper=1.57079632679 effort=10 velocity=1.0 -> lower=0 upper=1.57079632679 effort=100 velocity=1.0
- joint MFJ4: limit lower=-0.43633231299858238 upper=0.43633231299858238 effort=10 velocity=1.0 -> lower=-0.43633231299858238 upper=0.43633231299858238 effort=100 velocity=1.0
- joint RFJ1: limit lower=0 upper=1.57079632679 effort=10 velocity=1.0 -> lower=0 upper=1.57079632679 effort=100 velocity=1.0
- joint RFJ2: limit lower=0 upper=1.57079632679 effort=10 velocity=1.0 -> lower=0 upper=1.57079632679 effort=100 velocity=1.0
- joint RFJ3: limit lower=0 upper=1.57079632679 effort=10 velocity=1.0 -> lower=0 upper=1.57079632679 effort=100 velocity=1.0
- joint RFJ4: limit lower=-0.43633231299858238 upper=0.43633231299858238 effort=10 velocity=1.0 -> lower=-0.43633231299858238 upper=0.43633231299858238 effort=100 velocity=1.0
- joint THJ1: limit lower=0 upper=1.571 effort=10 velocity=1.0 -> lower=0 upper=1.571 effort=100 velocity=1.0
- joint THJ2: limit lower=-0.5237 upper=0.5237 effort=10 velocity=1.0 -> lower=-0.5237 upper=0.5237 effort=100 velocity=1.0
- joint THJ3: limit lower=-0.2618 upper=0.2618 effort=10 velocity=1.0 -> lower=-0.2618 upper=0.2618 effort=100 velocity=1.0
- joint THJ4: limit lower=0 upper=1.309 effort=10 velocity=1.0 -> lower=0 upper=1.309 effort=100 velocity=1.0
- joint THJ5: limit lower=-1.047 upper=1.047 effort=10 velocity=1.0 -> lower=-1.047 upper=1.047 effort=100 velocity=1.0

Commit message: Fixing the gazebo tactile sensors to work with stock gazebo

File: urdf/gazebo_shadowhand_standalone.urdf.xacro (robot description, xacro)
@@ -7,7 +7,12 @@
   <gazebo reference="ffdistal">
     <sensor type="contact" name="ffdistal_contact" >
+      <always_on>1</always_on>
+      <update_rate>1000.0</update_rate>
+      <contact>
+        <collision>ffdistal_collision</collision>
+        <topic>ffdistal_collision</topic>
+      </contact>
       <plugin name="ffdistal_gazebo_ros_bumper_controller" filename="libgazebo_ros_bumper.so">
-	<alwaysOn>true</alwaysOn>
-	<updateRate>100.0</updateRate>
+        <updateRate>100.0</updateRate>
 	<frameName>ffdistal</frameName>
 	<bumperTopicName>/sh/contacts/ff</bumperTopicName>
@@ -17,8 +22,13 @@
   </gazebo>
   <gazebo reference="mfdistal">
-    <sensor type="contact" name="mf_contact" >
-      <plugin name="mf_gazebo_ros_bumper_controller" filename="libgazebo_ros_bumper.so">
-	<alwaysOn>true</alwaysOn>
-	<updateRate>100.0</updateRate>
+    <sensor type="contact" name="mfdistal_contact" >
+      <always_on>1</always_on>
+      <update_rate>1000.0</update_rate>
+      <contact>
+        <collision>mfdistal_collision</collision>
+        <topic>mfdistal_collision</topic>
+      </contact>
+      <plugin name="mfdistal_gazebo_ros_bumper_controller" filename="libgazebo_ros_bumper.so">
+        <updateRate>100.0</updateRate>
 	<frameName>mfdistal</frameName>
 	<bumperTopicName>/sh/contacts/mf</bumperTopicName>
@@ -28,8 +38,13 @@
   </gazebo>
   <gazebo reference="rfdistal">
-    <sensor type="contact" name="mf_contact" >
-      <plugin name="mf_gazebo_ros_bumper_controller" filename="libgazebo_ros_bumper.so">
-	<alwaysOn>true</alwaysOn>
-	<updateRate>100.0</updateRate>
+    <sensor type="contact" name="rfdistal_contact" >
+      <always_on>1</always_on>
+      <update_rate>1000.0</update_rate>
+      <contact>
+        <collision>rfdistal_collision</collision>
+        <topic>rfdistal_collision</topic>
+      </contact>
+      <plugin name="rfdistal_gazebo_ros_bumper_controller" filename="libgazebo_ros_bumper.so">
+        <updateRate>100.0</updateRate>
 	<frameName>rfdistal</frameName>
 	<bumperTopicName>/sh/contacts/rf</bumperTopicName>
@@ -39,8 +54,13 @@
   </gazebo>
   <gazebo reference="lfdistal">
-    <sensor type="contact" name="lf_contact" >
-      <plugin name="lf_gazebo_ros_bumper_controller" filename="libgazebo_ros_bumper.so">
-	<alwaysOn>true</alwaysOn>
-	<updateRate>100.0</updateRate>
+    <sensor type="contact" name="lfdistal_contact" >
+      <always_on>1</always_on>
+      <update_rate>1000.0</update_rate>
+      <contact>
+        <collision>lfdistal_collision</collision>
+        <topic>lfdistal_collision</topic>
+      </contact>
+      <plugin name="lfdistal_gazebo_ros_bumper_controller" filename="libgazebo_ros_bumper.so">
+        <updateRate>100.0</updateRate>
 	<frameName>lfdistal</frameName>
 	<bumperTopicName>/sh/contacts/lf</bumperTopicName>
@@ -50,8 +70,13 @@
   </gazebo>
   <gazebo reference="thdistal">
-    <sensor type="contact" name="th_contact" >
-      <plugin name="th_gazebo_ros_bumper_controller" filename="libgazebo_ros_bumper.so">
-	<alwaysOn>true</alwaysOn>
-	<updateRate>100.0</updateRate>
+    <sensor type="contact" name="thdistal_contact" >
+      <always_on>1</always_on>
+      <update_rate>1000.0</update_rate>
+      <contact>
+        <collision>thdistal_collision</collision>
+        <topic>thdistal_collision</topic>
+      </contact>
+      <plugin name="thdistal_gazebo_ros_bumper_controller" filename="libgazebo_ros_bumper.so">
+        <updateRate>100.0</updateRate>
 	<frameName>thdistal</frameName>
 	<bumperTopicName>/sh/contacts/th</bumperTopicName>

Commit message: Fix LFJ5 and THJ5.

File: urdf/gazebo_shadowhand_standalone.urdf.xacro (robot description, xacro)
@@ -204,4 +204,12 @@
     </actuator>
   </transmission>
+  <transmission name="trans_lfj5">
+    <type>transmission_interface/SimpleTransmission</type>
+    <joint name="LFJ5"/>
+    <actuator name="motor_lfj5">
+      <hardwareInterface>EffortJointInterface</hardwareInterface>
+      <mechanicalReduction>1</mechanicalReduction>
+    </actuator>
+  </transmission>
   <transmission name="trans_thj1">
     <type>transmission_interface/SimpleTransmission</type>
@@ -232,4 +240,12 @@
     <joint name="THJ4"/>
     <actuator name="motor_thj4">
+      <hardwareInterface>EffortJointInterface</hardwareInterface>
+      <mechanicalReduction>1</mechanicalReduction>
+    </actuator>
+  </transmission>
+  <transmission name="trans_thj5">
+    <type>transmission_interface/SimpleTransmission</type>
+    <joint name="THJ5"/>
+    <actuator name="motor_thj5">
       <hardwareInterface>EffortJointInterface</hardwareInterface>
       <mechanicalReduction>1</mechanicalReduction>

Commit message: The GSC hand has ATI nanos on TH,FF,RF and PSTs on RF,LF

File: urdf/gazebo_shadowhand_standalone.urdf.xacro (robot description, xacro)
@@ -35,5 +35,5 @@
       </plugin>
     </sensor>
-    <material>Gazebo/Orange</material>
+    <material>Gazebo/Green</material>
   </gazebo>
   <gazebo reference="rfdistal">
@@ -67,5 +67,5 @@
       </plugin>
     </sensor>
-    <material>Gazebo/Orange</material>
+    <material>Gazebo/Green</material>
   </gazebo>
   <gazebo reference="thdistal">

File: urdf/shadowhand.urdf (robot description, URDF)
Before this commit: robot shadowhand, 30 links, 29 joints
Links:
- link lfdistal: geometry collision mesh filename=package://sr_grasp_description/meshes/F1.dae scale=0.1 0.1 0.1; visual mesh filename=package://sr_grasp_description/meshes/F1.dae scale=0.1 0.1 0.1
- link mfdistal: geometry collision mesh filename=package://sr_grasp_description/meshes/F1.dae scale=0.1 0.1 0.1; visual mesh filename=package://sr_grasp_description/meshes/F1.dae scale=0.1 0.1 0.1
