Commit message: using model from sr_description + our default position controllers

File: urdf/gazebo_shadowhand_standalone.urdf.xacro (robot description, xacro)
@@ -1,280 +1,3 @@
 <robot name="shadowhand" xmlns:xacro="http://www.ros.org/wiki/xacro">
-  <gazebo>
-    <plugin name="ros_control" filename="libgazebo_ros_control.so">
-      <robotNamespace>/rh</robotNamespace>
-    </plugin>
-  </gazebo>
-  <gazebo reference="ffdistal">
-    <sensor type="contact" name="ffdistal_contact" >
-      <always_on>1</always_on>
-      <update_rate>1000.0</update_rate>
-      <contact>
-        <collision>ffdistal_collision</collision>
-        <topic>ffdistal_collision</topic>
-      </contact>
-      <plugin name="ffdistal_gazebo_ros_bumper_controller" filename="libgazebo_ros_bumper.so">
-        <updateRate>100.0</updateRate>
-	<frameName>ffdistal</frameName>
-	<bumperTopicName>/rh/contacts/ff</bumperTopicName>
-      </plugin>
-    </sensor>
-    <material>Gazebo/Orange</material>
-  </gazebo>
-  <gazebo reference="mfdistal">
-    <sensor type="contact" name="mfdistal_contact" >
-      <always_on>1</always_on>
-      <update_rate>1000.0</update_rate>
-      <contact>
-        <collision>mfdistal_collision</collision>
-        <topic>mfdistal_collision</topic>
-      </contact>
-      <plugin name="mfdistal_gazebo_ros_bumper_controller" filename="libgazebo_ros_bumper.so">
-        <updateRate>100.0</updateRate>
-	<frameName>mfdistal</frameName>
-	<bumperTopicName>/rh/contacts/mf</bumperTopicName>
-      </plugin>
-    </sensor>
-    <material>Gazebo/Green</material>
-  </gazebo>
-  <gazebo reference="rfdistal">
-    <sensor type="contact" name="rfdistal_contact" >
-      <always_on>1</always_on>
-      <update_rate>1000.0</update_rate>
-      <contact>
-        <collision>rfdistal_collision</collision>
-        <topic>rfdistal_collision</topic>
-      </contact>
-      <plugin name="rfdistal_gazebo_ros_bumper_controller" filename="libgazebo_ros_bumper.so">
-        <updateRate>100.0</updateRate>
-	<frameName>rfdistal</frameName>
-	<bumperTopicName>/rh/contacts/rf</bumperTopicName>
-      </plugin>
-    </sensor>
-    <material>Gazebo/Orange</material>
-  </gazebo>
-  <gazebo reference="lfdistal">
-    <sensor type="contact" name="lfdistal_contact" >
-      <always_on>1</always_on>
-      <update_rate>1000.0</update_rate>
-      <contact>
-        <collision>lfdistal_collision</collision>
-        <topic>lfdistal_collision</topic>
-      </contact>
-      <plugin name="lfdistal_gazebo_ros_bumper_controller" filename="libgazebo_ros_bumper.so">
-        <updateRate>100.0</updateRate>
-	<frameName>lfdistal</frameName>
-	<bumperTopicName>/rh/contacts/lf</bumperTopicName>
-      </plugin>
-    </sensor>
-    <material>Gazebo/Green</material>
-  </gazebo>
-  <gazebo reference="thdistal">
-    <sensor type="contact" name="thdistal_contact" >
-      <always_on>1</always_on>
-      <update_rate>1000.0</update_rate>
-      <contact>
-        <collision>thdistal_collision</collision>
-        <topic>thdistal_collision</topic>
-      </contact>
-      <plugin name="thdistal_gazebo_ros_bumper_controller" filename="libgazebo_ros_bumper.so">
-        <updateRate>100.0</updateRate>
-	<frameName>thdistal</frameName>
-	<bumperTopicName>/rh/contacts/th</bumperTopicName>
-      </plugin>
-    </sensor>
-    <material>Gazebo/Orange</material>
-  </gazebo>
-  <transmission name="trans_wrj1">
-    <type>transmission_interface/SimpleTransmission</type>
-    <joint name="WRJ1"/>
-    <actuator name="motor_wrj1">
-      <hardwareInterface>EffortJointInterface</hardwareInterface>
-      <mechanicalReduction>1</mechanicalReduction>
-    </actuator>
-  </transmission>
-  <transmission name="trans_wrj2">
-    <type>transmission_interface/SimpleTransmission</type>
-    <joint name="WRJ2"/>
-    <actuator name="motor_wrj2">
-      <hardwareInterface>EffortJointInterface</hardwareInterface>
-      <mechanicalReduction>1</mechanicalReduction>
-    </actuator>
-  </transmission>
-  <transmission name="trans_ffj1">
-    <type>transmission_interface/SimpleTransmission</type>
-    <joint name="FFJ1"/>
-    <actuator name="motor_ffj1">
-      <hardwareInterface>EffortJointInterface</hardwareInterface>
-      <mechanicalReduction>1</mechanicalReduction>
-    </actuator>
-  </transmission>
-  <transmission name="trans_ffj2">
-    <type>transmission_interface/SimpleTransmission</type>
-    <joint name="FFJ2"/>
-    <actuator name="motor_ffj2">
-      <hardwareInterface>EffortJointInterface</hardwareInterface>
-      <mechanicalReduction>1</mechanicalReduction>
-    </actuator>
-  </transmission>
-  <transmission name="trans_ffj3">
-    <type>transmission_interface/SimpleTransmission</type>
-    <joint name="FFJ3"/>
-    <actuator name="motor_ffj3">
-      <hardwareInterface>EffortJointInterface</hardwareInterface>
-      <mechanicalReduction>1</mechanicalReduction>
-    </actuator>
-  </transmission>
-  <transmission name="trans_ffj4">
-    <type>transmission_interface/SimpleTransmission</type>
-    <joint name="FFJ4"/>
-    <actuator name="motor_ffj4">
-      <hardwareInterface>EffortJointInterface</hardwareInterface>
-      <mechanicalReduction>1</mechanicalReduction>
-    </actuator>
-  </transmission>
-  <transmission name="trans_mfj1">
-    <type>transmission_interface/SimpleTransmission</type>
-    <joint name="MFJ1"/>
-    <actuator name="motor_mfj1">
-      <hardwareInterface>EffortJointInterface</hardwareInterface>
-      <mechanicalReduction>1</mechanicalReduction>
-    </actuator>
-  </transmission>
-  <transmission name="trans_mfj2">
-    <type>transmission_interface/SimpleTransmission</type>
-    <joint name="MFJ2"/>
-    <actuator name="motor_mfj2">
-      <hardwareInterface>EffortJointInterface</hardwareInterface>
-      <mechanicalReduction>1</mechanicalReduction>
-    </actuator>
-  </transmission>
-  <transmission name="trans_mfj3">
-    <type>transmission_interface/SimpleTransmission</type>
-    <joint name="MFJ3"/>
-    <actuator name="motor_mfj3">
-      <hardwareInterface>EffortJointInterface</hardwareInterface>
-      <mechanicalReduction>1</mechanicalReduction>
-    </actuator>
-  </transmission>
-  <transmission name="trans_mfj4">
-    <type>transmission_interface/SimpleTransmission</type>
-    <joint name="MFJ4"/>
-    <actuator name="motor_mfj4">
-      <hardwareInterface>EffortJointInterface</hardwareInterface>
-      <mechanicalReduction>1</mechanicalReduction>
-    </actuator>
-  </transmission>
-  <transmission name="trans_rfj1">
-    <type>transmission_interface/SimpleTransmission</type>
-    <joint name="RFJ1"/>
-    <actuator name="motor_rfj1">
-      <hardwareInterface>EffortJointInterface</hardwareInterface>
-      <mechanicalReduction>1</mechanicalReduction>
-    </actuator>
-  </transmission>
-  <transmission name="trans_rfj2">
-    <type>transmission_interface/SimpleTransmission</type>
-    <joint name="RFJ2"/>
-    <actuator name="motor_rfj2">
-      <hardwareInterface>EffortJointInterface</hardwareInterface>
-      <mechanicalReduction>1</mechanicalReduction>
-    </actuator>
-  </transmission>
-  <transmission name="trans_rfj3">
-    <type>transmission_interface/SimpleTransmission</type>
-    <joint name="RFJ3"/>
-    <actuator name="motor_rfj3">
-      <hardwareInterface>EffortJointInterface</hardwareInterface>
-      <mechanicalReduction>1</mechanicalReduction>
-    </actuator>
-  </transmission>
-  <transmission name="trans_rfj4">
-    <type>transmission_interface/SimpleTransmission</type>
-    <joint name="RFJ4"/>
-    <actuator name="motor_rfj4">
-      <hardwareInterface>EffortJointInterface</hardwareInterface>
-      <mechanicalReduction>1</mechanicalReduction>
-    </actuator>
-  </transmission>
-  <transmission name="trans_lfj1">
-    <type>transmission_interface/SimpleTransmission</type>
-    <joint name="LFJ1"/>
-    <actuator name="motor_lfj1">
-      <hardwareInterface>EffortJointInterface</hardwareInterface>
-      <mechanicalReduction>1</mechanicalReduction>
-    </actuator>
-  </transmission>
-  <transmission name="trans_lfj2">
-    <type>transmission_interface/SimpleTransmission</type>
-    <joint name="LFJ2"/>
-    <actuator name="motor_lfj2">
-      <hardwareInterface>EffortJointInterface</hardwareInterface>
-      <mechanicalReduction>1</mechanicalReduction>
-    </actuator>
-  </transmission>
-  <transmission name="trans_lfj3">
-    <type>transmission_interface/SimpleTransmission</type>
-    <joint name="LFJ3"/>
-    <actuator name="motor_lfj3">
-      <hardwareInterface>EffortJointInterface</hardwareInterface>
-      <mechanicalReduction>1</mechanicalReduction>
-    </actuator>
-  </transmission>
-  <transmission name="trans_lfj4">
-    <type>transmission_interface/SimpleTransmission</type>
-    <joint name="LFJ4"/>
-    <actuator name="motor_lfj4">
-      <hardwareInterface>EffortJointInterface</hardwareInterface>
-      <mechanicalReduction>1</mechanicalReduction>
-    </actuator>
-  </transmission>
-  <transmission name="trans_lfj5">
-    <type>transmission_interface/SimpleTransmission</type>
-    <joint name="LFJ5"/>
-    <actuator name="motor_lfj5">
-      <hardwareInterface>EffortJointInterface</hardwareInterface>
-      <mechanicalReduction>1</mechanicalReduction>
-    </actuator>
-  </transmission>
-  <transmission name="trans_thj1">
-    <type>transmission_interface/SimpleTransmission</type>
-    <joint name="THJ1"/>
-    <actuator name="motor_thj1">
-      <hardwareInterface>EffortJointInterface</hardwareInterface>
-      <mechanicalReduction>1</mechanicalReduction>
-    </actuator>
-  </transmission>
-  <transmission name="trans_thj2">
-    <type>transmission_interface/SimpleTransmission</type>
-    <joint name="THJ2"/>
-    <actuator name="motor_thj2">
-      <hardwareInterface>EffortJointInterface</hardwareInterface>
-      <mechanicalReduction>1</mechanicalReduction>
-    </actuator>
-  </transmission>
-  <transmission name="trans_thj3">
-    <type>transmission_interface/SimpleTransmission</type>
-    <joint name="THJ3"/>
-    <actuator name="motor_thj3">
-      <hardwareInterface>EffortJointInterface</hardwareInterface>
-      <mechanicalReduction>1</mechanicalReduction>
-    </actuator>
-  </transmission>
-  <transmission name="trans_thj4">
-    <type>transmission_interface/SimpleTransmission</type>
-    <joint name="THJ4"/>
-    <actuator name="motor_thj4">
-      <hardwareInterface>EffortJointInterface</hardwareInterface>
-      <mechanicalReduction>1</mechanicalReduction>
-    </actuator>
-  </transmission>
-  <transmission name="trans_thj5">
-    <type>transmission_interface/SimpleTransmission</type>
-    <joint name="THJ5"/>
-    <actuator name="motor_thj5">
-      <hardwareInterface>EffortJointInterface</hardwareInterface>
-      <mechanicalReduction>1</mechanicalReduction>
-    </actuator>
-  </transmission>
   <!-- adding fixed link to world for the hand not to fall -->
   <link name="world"/>
@@ -283,5 +6,8 @@
     <child link="forearm"/>
   </joint>
-  <!-- loading the shadow hand -->
-  <xacro:include filename="$(find sr_grasp_description)/urdf/shadowhand.urdf" />
+  <xacro:include filename="$(find sr_description)/materials.urdf.xacro" />
+  <xacro:include filename="$(find sr_description)/hand/xacro/full_hand_motor.urdf.xacro" />
+  <xacro:include filename="$(find sr_description)/other/xacro/gazebo/gazebo.urdf.xacro" />
+  <xacro:shadowhand_motor>
+  </xacro:shadowhand_motor>
 </robot>

Commit message: spawning a kinect in simu, fixed rviz visualisation problem as well (bad hand position)

File: urdf/gazebo_shadowhand_standalone.urdf.xacro (robot description, xacro)
@@ -1,3 +1,9 @@
 <robot name="shadowhand" xmlns:xacro="http://www.ros.org/wiki/xacro">
+  <property name="cam_px" value="-0.3" />
+  <property name="cam_py" value="0.0" />
+  <property name="cam_pz" value="1.1" />
+  <property name="cam_or" value="0.0" />
+  <property name="cam_op" value="0.0" />
+  <property name="cam_oy" value="0.0" />
   <!-- adding fixed link to world for the hand not to fall -->
   <link name="world"/>
@@ -5,4 +11,5 @@
     <parent link="world"/>
     <child link="forearm"/>
+    <origin xyz="0.8 0.0 1.1" rpy="1.57 -1.57 -1.57"/>
   </joint>
   <xacro:include filename="$(find sr_description)/materials.urdf.xacro" />
@@ -11,3 +18,124 @@
   <xacro:shadowhand_motor>
   </xacro:shadowhand_motor>
+  <joint name="camera_rgb_joint" type="fixed">
+    <origin xyz="${cam_px} ${cam_py} ${cam_pz}" rpy="${cam_or} ${cam_op} ${cam_oy}"/>
+    <parent link="world"/>
+    <child link="camera_rgb_frame" />
+  </joint>
+  <link name="camera_rgb_frame">
+    <inertial>
+      <mass value="0.001" />
+      <origin xyz="0 0 0" />
+      <inertia ixx="0.0001" ixy="0.0" ixz="0.0"
+               iyy="0.0001" iyz="0.0"
+               izz="0.0001" />
+    </inertial>
+  </link>
+  <joint name="camera_rgb_optical_joint" type="fixed">
+    <origin xyz="0 0 0" rpy="${-M_PI/2} 0 ${-M_PI/2}" />
+    <parent link="camera_rgb_frame" />
+    <child link="camera_rgb_optical_frame" />
+  </joint>
+  <link name="camera_rgb_optical_frame">
+    <inertial>
+      <mass value="0.001" />
+      <origin xyz="0 0 0" />
+      <inertia ixx="0.0001" ixy="0.0" ixz="0.0"
+               iyy="0.0001" iyz="0.0"
+               izz="0.0001" />
+    </inertial>
+  </link>
+  <joint name="camera_joint" type="fixed">
+    <origin xyz="-0.031 ${-cam_py} -0.016" rpy="0 0 0"/>
+    <parent link="camera_rgb_frame"/>
+    <child link="camera_link"/>
+  </joint>
+  <link name="camera_link">
+    <visual>
+      <origin xyz="0 0 0" rpy="0 0 ${M_PI/2}"/>
+      <geometry>
+        <mesh filename="package://sr_grasp_gazebo/model/kinect.dae"/>
+      </geometry>
+    </visual>
+    <collision>
+      <origin xyz="0.0 0.0 0.0" rpy="0 0 0"/>
+      <geometry>
+	<box size="0.07271 0.27794 0.073"/>
+      </geometry>
+    </collision>
+    <inertial>
+      <mass value="0.001" />
+      <origin xyz="0 0 0" />
+      <inertia ixx="0.0001" ixy="0.0" ixz="0.0"
+               iyy="0.0001" iyz="0.0"
+               izz="0.0001" />
+    </inertial>
+  </link>
+  <!-- The fixed joints & links below are usually published by static_transformers launched by the OpenNi launch
+       files. However, for Gazebo simulation we need them, so we add them here.
+       (Hence, don't publish them additionally!) -->
+  <joint name="camera_depth_joint" type="fixed">
+    <origin xyz="0 ${2 * -cam_py} 0" rpy="0 0 0" />
+    <parent link="camera_rgb_frame" />
+    <child link="camera_depth_frame" />
+  </joint>
+  <link name="camera_depth_frame">
+    <inertial>
+      <mass value="0.001" />
+      <origin xyz="0 0 0" />
+      <inertia ixx="0.0001" ixy="0.0" ixz="0.0"
+               iyy="0.0001" iyz="0.0"
+               izz="0.0001" />
+    </inertial>
+  </link>
+  <joint name="camera_depth_optical_joint" type="fixed">
+    <origin xyz="0 0 0" rpy="${-M_PI/2} 0 ${-M_PI/2}" />
+    <parent link="camera_depth_frame" />
+    <child link="camera_depth_optical_frame" />
+  </joint>
+  <link name="camera_depth_optical_frame">
+    <inertial>
+      <mass value="0.001" />
+      <origin xyz="0 0 0" />
+      <inertia ixx="0.0001" ixy="0.0" ixz="0.0"
+               iyy="0.0001" iyz="0.0"
+               izz="0.0001" />
+    </inertial>
+  </link>
+  <gazebo reference="camera_link">
+    <sensor type="depth" name="camera">
+      <always_on>true</always_on>
+      <update_rate>20.0</update_rate>
+      <camera>
+        <horizontal_fov>${60.0*M_PI/180.0}</horizontal_fov>
+        <image>
+          <format>R8G8B8</format>
+          <width>640</width>
+          <height>480</height>
+        </image>
+        <clip>
+          <near>0.05</near>
+          <far>8.0</far>
+        </clip>
+      </camera>
+      <plugin name="kinect_camera_controller" filename="libgazebo_ros_openni_kinect.so">
+        <cameraName>camera</cameraName>
+        <alwaysOn>true</alwaysOn>
+        <updateRate>10</updateRate>
+        <imageTopicName>rgb/image_raw</imageTopicName>
+        <depthImageTopicName>depth/image_raw</depthImageTopicName>
+        <pointCloudTopicName>depth/points</pointCloudTopicName>
+        <cameraInfoTopicName>rgb/camera_info</cameraInfoTopicName>
+        <depthImageCameraInfoTopicName>depth/camera_info</depthImageCameraInfoTopicName>
+        <frameName>camera_depth_optical_frame</frameName>
+        <baseline>0.1</baseline>
+        <distortion_k1>0.0</distortion_k1>
+        <distortion_k2>0.0</distortion_k2>
+        <distortion_k3>0.0</distortion_k3>
+        <distortion_t1>0.0</distortion_t1>
+        <distortion_t2>0.0</distortion_t2>
+        <pointCloudCutoff>0.4</pointCloudCutoff>
+      </plugin>
+    </sensor>
+  </gazebo>
 </robot>

Commit message: adding rviz config for debugging + instructions

File: urdf/gazebo_shadowhand_standalone.urdf.xacro (robot description, xacro)
@@ -18,124 +18,3 @@
   <xacro:shadowhand_motor>
   </xacro:shadowhand_motor>
-  <joint name="camera_rgb_joint" type="fixed">
-    <origin xyz="${cam_px} ${cam_py} ${cam_pz}" rpy="${cam_or} ${cam_op} ${cam_oy}"/>
-    <parent link="world"/>
-    <child link="camera_rgb_frame" />
-  </joint>
-  <link name="camera_rgb_frame">
-    <inertial>
-      <mass value="0.001" />
-      <origin xyz="0 0 0" />
-      <inertia ixx="0.0001" ixy="0.0" ixz="0.0"
-               iyy="0.0001" iyz="0.0"
-               izz="0.0001" />
-    </inertial>
-  </link>
-  <joint name="camera_rgb_optical_joint" type="fixed">
-    <origin xyz="0 0 0" rpy="${-M_PI/2} 0 ${-M_PI/2}" />
-    <parent link="camera_rgb_frame" />
-    <child link="camera_rgb_optical_frame" />
-  </joint>
-  <link name="camera_rgb_optical_frame">
-    <inertial>
-      <mass value="0.001" />
-      <origin xyz="0 0 0" />
-      <inertia ixx="0.0001" ixy="0.0" ixz="0.0"
-               iyy="0.0001" iyz="0.0"
-               izz="0.0001" />
-    </inertial>
-  </link>
-  <joint name="camera_joint" type="fixed">
-    <origin xyz="-0.031 ${-cam_py} -0.016" rpy="0 0 0"/>
-    <parent link="camera_rgb_frame"/>
-    <child link="camera_link"/>
-  </joint>
-  <link name="camera_link">
-    <visual>
-      <origin xyz="0 0 0" rpy="0 0 ${M_PI/2}"/>
-      <geometry>
-        <mesh filename="package://sr_grasp_gazebo/model/kinect.dae"/>
-      </geometry>
-    </visual>
-    <collision>
-      <origin xyz="0.0 0.0 0.0" rpy="0 0 0"/>
-      <geometry>
-	<box size="0.07271 0.27794 0.073"/>
-      </geometry>
-    </collision>
-    <inertial>
-      <mass value="0.001" />
-      <origin xyz="0 0 0" />
-      <inertia ixx="0.0001" ixy="0.0" ixz="0.0"
-               iyy="0.0001" iyz="0.0"
-               izz="0.0001" />
-    </inertial>
-  </link>
-  <!-- The fixed joints & links below are usually published by static_transformers launched by the OpenNi launch
-       files. However, for Gazebo simulation we need them, so we add them here.
-       (Hence, don't publish them additionally!) -->
-  <joint name="camera_depth_joint" type="fixed">
-    <origin xyz="0 ${2 * -cam_py} 0" rpy="0 0 0" />
-    <parent link="camera_rgb_frame" />
-    <child link="camera_depth_frame" />
-  </joint>
-  <link name="camera_depth_frame">
-    <inertial>
-      <mass value="0.001" />
-      <origin xyz="0 0 0" />
-      <inertia ixx="0.0001" ixy="0.0" ixz="0.0"
-               iyy="0.0001" iyz="0.0"
-               izz="0.0001" />
-    </inertial>
-  </link>
-  <joint name="camera_depth_optical_joint" type="fixed">
-    <origin xyz="0 0 0" rpy="${-M_PI/2} 0 ${-M_PI/2}" />
-    <parent link="camera_depth_frame" />
-    <child link="camera_depth_optical_frame" />
-  </joint>
-  <link name="camera_depth_optical_frame">
-    <inertial>
-      <mass value="0.001" />
-      <origin xyz="0 0 0" />
-      <inertia ixx="0.0001" ixy="0.0" ixz="0.0"
-               iyy="0.0001" iyz="0.0"
-               izz="0.0001" />
-    </inertial>
-  </link>
-  <gazebo reference="camera_link">
-    <sensor type="depth" name="camera">
-      <always_on>true</always_on>
-      <update_rate>20.0</update_rate>
-      <camera>
-        <horizontal_fov>${60.0*M_PI/180.0}</horizontal_fov>
-        <image>
-          <format>R8G8B8</format>
-          <width>640</width>
-          <height>480</height>
-        </image>
-        <clip>
-          <near>0.05</near>
-          <far>8.0</far>
-        </clip>
-      </camera>
-      <plugin name="kinect_camera_controller" filename="libgazebo_ros_openni_kinect.so">
-        <cameraName>camera</cameraName>
-        <alwaysOn>true</alwaysOn>
-        <updateRate>10</updateRate>
-        <imageTopicName>rgb/image_raw</imageTopicName>
-        <depthImageTopicName>depth_registered/image_raw</depthImageTopicName>
-        <pointCloudTopicName>depth_registered/points</pointCloudTopicName>
-        <cameraInfoTopicName>rgb/camera_info</cameraInfoTopicName>
-        <depthImageCameraInfoTopicName>depth_registered/camera_info</depthImageCameraInfoTopicName>
-        <frameName>camera_depth_optical_frame</frameName>
-        <baseline>0.1</baseline>
-        <distortion_k1>0.0</distortion_k1>
-        <distortion_k2>0.0</distortion_k2>
-        <distortion_k3>0.0</distortion_k3>
-        <distortion_t1>0.0</distortion_t1>
-        <distortion_t2>0.0</distortion_t2>
-        <pointCloudCutoff>0.4</pointCloudCutoff>
-      </plugin>
-    </sensor>
-  </gazebo>
 </robot>
