Commit message: Updating references to hand mesh locations

File: sr_grasp_description/urdf/shadowhand_motor_ellipsoid.orig.urdf (robot description, URDF)
Before this commit: robot shadowhand_motor, 30 links, 29 joints
Links:
- link ffdistal: geometry collision mesh filename=package://sr_description/meshes/hand/distal_ellipsoid.dae scale=0.001 0.001 0.001; visual mesh filename=package://sr_description/meshes/hand/distal_ellipsoid.dae scale=0.001 0.001 0.001
- link ffknuckle: geometry collision box size=0.005 0.005 0.005; visual mesh filename=package://sr_description/meshes/hand/knuckle.dae scale=0.001 0.001 0.001
- link ffmiddle: geometry collision box size=0.008 0.008 0.015; visual mesh filename=package://sr_description/meshes/hand/F2.dae scale=0.001 0.001 0.001
- link ffproximal: geometry collision box size=0.008 0.008 0.04; visual mesh filename=package://sr_description/meshes/hand/F3.dae scale=0.001 0.001 0.001
- link forearm: geometry collision cylinder length=0.180 radius=0.06; visual mesh filename=package://sr_description/meshes/hand/forearm.dae scale=0.001 0.001 0.001
- link lfdistal: geometry collision mesh filename=package://sr_description/meshes/hand/distal_ellipsoid.dae scale=0.001 0.001 0.001; visual mesh filename=package://sr_description/meshes/hand/distal_ellipsoid.dae scale=0.001 0.001 0.001
- link lfknuckle: geometry collision box size=0.005 0.005 0.005; visual mesh filename=package://sr_description/meshes/hand/knuckle.dae scale=0.001 0.001 0.001
- link lfmetacarpal: geometry collision box size=0.008 0.008 0.03; visual mesh filename=package://sr_description/meshes/hand/lfmetacarpal.dae scale=0.001 0.001 0.001
- link lfmiddle: geometry collision box size=0.008 0.008 0.015; visual mesh filename=package://sr_description/meshes/hand/F2.dae scale=0.001 0.001 0.001
- link lfproximal: geometry collision box size=0.008 0.008 0.04; visual mesh filename=package://sr_description/meshes/hand/F3.dae scale=0.001 0.001 0.001
- link mfdistal: geometry collision mesh filename=package://sr_description/meshes/hand/distal_ellipsoid.dae scale=0.001 0.001 0.001; visual mesh filename=package://sr_description/meshes/hand/distal_ellipsoid.dae scale=0.001 0.001 0.001
- link mfknuckle: geometry collision box size=0.005 0.005 0.005; visual mesh filename=package://sr_description/meshes/hand/knuckle.dae scale=0.001 0.001 0.001
- link mfmiddle: geometry collision box size=0.008 0.008 0.015; visual mesh filename=package://sr_description/meshes/hand/F2.dae scale=0.001 0.001 0.001
- link mfproximal: geometry collision box size=0.008 0.008 0.04; visual mesh filename=package://sr_description/meshes/hand/F3.dae scale=0.001 0.001 0.001
- link palm: geometry collision box size=0.05 0.02 0.07; visual mesh filename=package://sr_description/meshes/hand/palm.dae scale=0.001 0.001 0.001
- link rfdistal: geometry collision mesh filename=package://sr_description/meshes/hand/distal_ellipsoid.dae scale=0.001 0.001 0.001; visual mesh filename=package://sr_description/meshes/hand/distal_ellipsoid.dae scale=0.001 0.001 0.001
- link rfknuckle: geometry collision box size=0.005 0.005 0.005; visual mesh filename=package://sr_description/meshes/hand/knuckle.dae scale=0.001 0.001 0.001
- link rfmiddle: geometry collision box size=0.008 0.008 0.015; visual mesh filename=package://sr_description/meshes/hand/F2.dae scale=0.001 0.001 0.001
- link rfproximal: geometry collision box size=0.008 0.008 0.04; visual mesh filename=package://sr_description/meshes/hand/F3.dae scale=0.001 0.001 0.001
- link thdistal: geometry collision mesh filename=package://sr_description/meshes/hand/distal_ellipsoid.dae scale=0.001 0.001 0.001; visual mesh filename=package://sr_description/meshes/hand/distal_ellipsoid.dae scale=0.001 0.001 0.001
- link thmiddle: geometry collision box size=0.008 0.008 0.015; visual mesh filename=package://sr_description/meshes/hand/TH2_z.dae scale=0.001 0.001 0.001
- link thproximal: geometry collision box size=0.008 0.008 0.020; visual mesh filename=package://sr_description/meshes/hand/TH3_z.dae scale=0.001 0.001 0.001
- link wrist: geometry collision box size=0.02 0.02 0.02; visual mesh filename=package://sr_description/meshes/hand/wrist.dae scale=0.001 0.001 0.001
